Commit message: foxy fixes modern cmake find cuda set common yaml parameters to our needs

File: zed_wrapper/urdf/zed2.urdf (robot description, URDF)
Before this commit: robot zed2_camera, 6 links, 5 joints
Links:
- removed link base_link
- added link zed2_base_link
Joints:
- joint zed2_camera_center_joint: parent base_link -> zed2_base_link
